Commit message: updates

File: husky-humble/husky_description/urdf/husky.urdf.xacro (robot description, xacro)
@@ -18,5 +18,5 @@
     <visual>
       <geometry>
-        <box size="0.1 0.05 0.05"/>
+        <box size="0.05 0.1 0.05"/>
       </geometry>
       <material name="Gray">
@@ -33,5 +33,5 @@
     <parent link="base_link"/>
     <child link="realsense_link"/>
-    <origin xyz="0.2 0 0.5" rpy="0 0 0"/>
+    <origin xyz="0.4 0 0.28" rpy="0 0 0"/>
   </joint>
   <!-- Camera sensor plugin for RGB camera -->
